Commit message: Make robot walk using joint controller and all legs; initial working gait walking weirdly

File: go2_description/gz/gz.xacro (robot description, xacro)
@@ -13,5 +13,5 @@
       <sensor name="imu_sensor" type="imu">
         <always_on>1</always_on>
-        <update_rate>4</update_rate>
+        <update_rate>50.0</update_rate>
         <visualize>true</visualize>
         <topic>imu</topic>

File: go2_description/urdf/torso.xacro (robot description, xacro)
@@ -4,4 +4,5 @@
     <!-- World frame -->
     <!-- <link name="world"/>  -->
+     <!-- <link name="odom"/>  -->
     <!-- <xacro:if value="${simulation}">
       <xacro:if value="${fixed_base}">
@@ -16,10 +17,9 @@
     <!-- <xacro:unless value="${fixed_base}"> -->
       <!-- <link name="odom"/> -->
-<!--
-      <joint name="world_to_odom" type="fixed">
+      <!-- <joint name="world_to_odom" type="fixed">
         <parent link="world"/>
-        <child link="odom"/>
-      </joint>
-      <joint name="odom_to_base" type="fixed">
+        <child link="base_link"/>
+      </joint> -->
+      <!-- <joint name="odom_to_base" type="fixed">
         <parent link="odom"/>
         <child link="base_link"/>
