Commit message: ekf filter added-position not working

File: go2_description/urdf/torso.xacro (robot description, xacro)
@@ -3,5 +3,5 @@
     <xacro:macro name="torso" params="simulation fixed_base">
     <!-- World frame -->
-    <link name="world"/>
+    <!-- <link name="world"/>  -->
     <!-- <xacro:if value="${simulation}">
       <xacro:if value="${fixed_base}">
@@ -15,5 +15,6 @@
     <!-- Movable base in simulation OR real robot -->
     <!-- <xacro:unless value="${fixed_base}"> -->
-      <link name="odom"/>
+      <!-- <link name="odom"/> -->
+<!--
       <joint name="world_to_odom" type="fixed">
         <parent link="world"/>
@@ -23,5 +24,5 @@
         <parent link="odom"/>
         <child link="base_link"/>
-      </joint>
+      </joint> -->
     <!-- </xacro:unless> -->
     <!-- Base link -->

Commit message: updated launch and xacro files

File: go2_description/urdf/torso.xacro (robot description, xacro)
@@ -2,10 +2,14 @@
 <robot xmlns:xacro="http://ros.org/wiki/xacro">
     <xacro:macro name="torso" params="simulation fixed_base">
-    <link name="world" />
+    <xacro:if value="$(arg fixed_base)">
+      <link name="world" />
+    </xacro:if>
     <link name="odom"/>
-    <joint name="world_to_odom" type="fixed">
-      <parent link="world"/>
-      <child link="odom"/>
-    </joint>
+    <xacro:if value="$(arg fixed_base)">
+      <joint name="world_to_odom" type="fixed">
+        <parent link="world"/>
+        <child link="odom"/>
+      </joint>
+    </xacro:if>
     <joint name="odom_to_base" type="fixed">
       <parent link="odom"/>
